File: hardware/VBC.sch (KiCad schematic (older format))
At the start: 5 parts, among them K1 RELAY_Metaltex, P1 CONN_01X01, U1 TS5A21366, U2 TS5A21366

Commit message: updated hardware files
Parts:
- added C1: Conn_SMA_90graus, Connectors:SMA_THT_Jack_Straight, symbol Conn_SMA_90graus
- added J1: Jack-DC, Connectors:BARREL_JACK, symbol Jack-DC
- added J2: USB_OTG, Connectors:USB_Micro-B, symbol USB_OTG
- added J3: 6P6C, Connectors:RJ12_E, symbol 6P6C
- added J4: Conn_01x02, Connectors_Terminal_Blocks:TerminalBlock_Altech_AK300-2_P5.00mm, symbol Conn_01x02
- added J5, J6, J7, J8: RJ11, Controle:RJ11, symbol RJ11
- added J9: USB_A, Connectors:USB_A, symbol USB_A
- added K2, K3, K4: RELAY_Metaltex, Relays_THT:Relay_DPDT_Omron_G5V-2, symbol RELAY_Metaltex
- added Q1, Q2, Q3, Q4: BC817, TO_SOT_Packages_SMD:SOT-23, symbol BC817
- added R1, R2, R3, R4, R5, R6: R, Resistors_SMD:R_0805_HandSoldering, symbol R
- K1: footprint (none) -> Relays_THT:Relay_DPDT_Omron_G5V-2
Connections:
- net VCC: now reaches K1.1
- net VCC: now also J1.1, K2.1, K3.1, K4.1
- net at K1.16: now also Q3.3 (C)
- net +24V: now reaches K1.4 (C1)
- net +24V: now also J4.1 (Pin_1), K2.4 (C1), K3.4 (C1), K4.4 (C1)
- net at K1.6 (R1): now also J7.2
- net at K1.8 (T1): now also J7.1
- new net: Q3.1 (B), R3.2
- new net: Q1.1 (B), R1.2
- new net: K2.16, Q1.3 (C)
- new net: J5.2, K2.6 (R1)
- new net: J5.1, K2.8 (T1)
- new net: Q4.1 (B), R4.2
- new net: K4.16, Q4.3 (C)
- new net: J8.2, K4.6 (R1)
- new net: J8.1, K4.8 (T1)
- new net: Q2.1 (B), R2.2
- new net: K3.16, Q2.3 (C)
- new net: J6.2, K3.6 (R1)
- new net: J6.1, K3.8 (T1)
- new net: C1.1, R5.1
- new net: J2.1 (VBUS), J9.1 (VBUS)
- new net: J2.2 (D-), J9.2 (D-)
- new net: J2.3 (D+), J9.3 (D+)
- new net AIn_BBB: R5.2, R6.1
- new net BBB_p?: R1.1, R2.1, R3.1, R4.1
- new net GND: C1.2, J1.2, J2.5 (GND), J2.6 (Shield), J9.4 (GND), J9.5 (Shield), Q1.2 (E), Q2.2 (E), Q3.2 (E), Q4.2 (E), R6.2
Other:
- moved on the sheet: Beagle1A, Beagle1B, K1, P1, U1, U2
