File: hardware/kicad/VBC.kicad_pcb (KiCad board)
At the start: 2 copper layers, 160 x 100 mm, 37 parts, among them J1 Conn_01x01, J10 Conn_01x01, J2 USB_OTG, J3 RJ25, J4 Conn_01x02, J5 RJ11, J6 RJ11, J7 RJ11, J8 RJ11, J9 USB_A, K1 RELAY_Metaltex, K2 RELAY_Metaltex, K3 RELAY_Metaltex, K4 RELAY_Metaltex, P1 CONN_01X01, Q1 BC817, Q2 BC817, Q3 BC817, Q4 BC817, U1 TS5A21366, U2 TS5A21366, U3 LT3080

Commit message: added relay LED status in schematic
Parts:
- removed U1, U2: TS5A21366, Controle:VSSOP-8

Commit message: new hardware version
Parts:
- removed U3: LT3080, TO_SOT_Packages_SMD:SOT-223
- added D10, D11, D12, D9: LED red, LEDs:LED_0805_HandSoldering, F.Cu at (136.9, 148.3)
- added D5, D6, D7, D8: LED green, LEDs:LED_0805_HandSoldering, F.Cu at (136.9, 148.3)
- added R10, R11, R12, R13, R14, R15, R16, R17, R18, R19, R20, R21, R22, R23, R24: 4k7, Resistors_SMD:R_0805_HandSoldering, F.Cu at (136.9, 148.3)
- added R30: 4k7, Resistors_SMD:R_0805, F.Cu at (136.9, 148.3)
- C1, J5, J6, J7, J8: moved to B.Cu
- J2: moved to F.Cu
- moved J1 98.4 mm to (124.2, 130.9), turned to 180 degrees
- moved J4 79.6 mm to (123.3, 51.2), turned to 90 degrees
- moved J9 46.1 mm to (69.4, 107.2)
- moved C1 9.78 mm to (219.4, 74.5)
- moved J2 4.45 mm to (64.0, 80.5)
- turned J5 to 270 degrees
- turned J6 to 270 degrees
- turned J7 to 270 degrees
- turned J8 to 270 degrees
Connections:
- net /K2_P11 renamed Net-(J5-Pad4)
- net /K2_P6 renamed Net-(D5-Pad2)
- net /K2_P8 renamed Net-(D9-Pad2)
- net /K2_P9 renamed Net-(J5-Pad3)
- net /K4_P11 renamed Net-(J8-Pad4)
- net /K4_P6 renamed Net-(D8-Pad2)
- net /K4_P8 renamed Net-(D12-Pad2)
- net /K4_P9 renamed Net-(J8-Pad3)
- Beagle1 pad C3: Net-(Beagle1-PadC3) -> /3.3V_BBB
- J3 pad 1: /VAT_P1 -> /3.3V_BBB
- J3 pad 6: /VAT_P6 -> /3.3V_BBB
- J6 pad 1: /K3_P8 -> Net-(D10-Pad2)
- J6 pad 2: /K3_P6 -> Net-(D6-Pad2)
- J6 pad 3: /K3_P9 -> Net-(J6-Pad3)
- J6 pad 4: /K3_P11 -> Net-(J6-Pad4)
- J7 pad 1: /K1_P8 -> Net-(D11-Pad2)
- J7 pad 2: /K1_P6 -> Net-(D7-Pad2)
- J7 pad 3: /K1_P9 -> Net-(J7-Pad3)
- J7 pad 4: /K1_P11 -> Net-(J7-Pad4)
- K1 pad 11: /K1_P11 -> Net-(J6-Pad4)
- K1 pad 6: /K1_P6 -> Net-(D6-Pad2)
- K1 pad 8: /K1_P8 -> Net-(D10-Pad2)
- K1 pad 9: /K1_P9 -> Net-(J6-Pad3)
- K3 pad 11: /K3_P11 -> Net-(J7-Pad4)
- K3 pad 6: /K3_P6 -> Net-(D7-Pad2)
- K3 pad 8: /K3_P8 -> Net-(D11-Pad2)
- K3 pad 9: /K3_P9 -> Net-(J7-Pad3)
Routing:
- net Net-(J6-Pad4): track 0.00 -> 141.9 mm
- net /3.3V_BBB: track 0.00 -> 120.7 mm
- net GND: track 154.4 -> 48.1 mm, vias 2 -> 1
- net (no net): track 0.00 -> 105.1 mm, vias 0 -> 1
- net /K1_P11: track 78.8 -> 0.00 mm
- net Net-(J7-Pad4): track 0.00 -> 77.4 mm
- net /K3_P11: track 74.2 -> 0.00 mm
- net /K1_P9: track 69.7 -> 0.00 mm
- net Net-(J6-Pad3): track 0.00 -> 66.4 mm
- net /K3_P9: track 66.0 -> 0.00 mm
- net /VAT_P1: track 63.7 -> 0.00 mm
- net /K1_P8: track 57.7 -> 0.00 mm
- net Net-(D10-Pad2): track 0.00 -> 57.7 mm
- net /VAT_P6: track 56.9 -> 0.00 mm
- net Net-(D6-Pad2): track 0.00 -> 53.3 mm
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Other:
- board size 160 x 100 mm -> 160 x 100.1 mm

Commit message: new hardware version
Parts:
- removed R9: 330K, Resistors_SMD:R_0805
- D10, D11, D12, D5, D6, D7, D8, D9, J3, J4, Q1, Q2, Q3, Q4, R10, R11, R12, R13, R14, R15, R16, R17, R18, R19, R20, R21, R22, R23, R24: moved to B.Cu
- R1, R2, R3, R30, R4: footprint Resistors_SMD:R_0805 -> Resistors_SMD:R_0805_HandSoldering; moved to B.Cu
- R5, R6, R7, R8: footprint Resistors_SMD:R_0805 -> Resistors_SMD:R_0805_HandSoldering
- moved R20 102.0 mm to (181.8, 56.6)
- moved R24 97.1 mm to (181.9, 62.2)
- moved D12 96.8 mm to (175.2, 59.3), turned to 180 degrees
- moved R18 93.1 mm to (154.5, 56.9)
- moved R13 92.4 mm to (181.9, 67.6)
- moved D8 91.7 mm to (175.1, 64.9), turned to 180 degrees
- moved D10 89.9 mm to (148.5, 59.1), turned to 180 degrees
- moved R21 88.0 mm to (154.5, 62.0)
- moved R17 87.8 mm to (182.0, 72.8)
- moved D6 84.7 mm to (148.6, 64.4), turned to 180 degrees
- moved R10 82.2 mm to (154.7, 68.0)
- moved R14 77.0 mm to (154.9, 73.3)
- moved R19 67.7 mm to (188.5, 104.4)
- moved R22 64.7 mm to (188.4, 109.2)
- moved R11 61.6 mm to (188.4, 114.3)
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- renumbered J7 to J6, J6 to J7
Connections:
- Beagle1 pad C3: /3.3V_BBB -> Net-(Beagle1-PadC3)
- Beagle1 pad C4: Net-(Beagle1-PadC4) -> /3.3V_BBB
- J6 pad 1: Net-(D11-Pad2) -> Net-(D10-Pad2)
- J6 pad 2: Net-(D7-Pad2) -> Net-(D6-Pad2)
- J6 pad 3: Net-(J7-Pad3) -> Net-(J6-Pad3)
- J6 pad 4: Net-(J7-Pad4) -> Net-(J6-Pad4)
- J7 pad 1: Net-(D10-Pad2) -> Net-(D11-Pad2)
- J7 pad 2: Net-(D6-Pad2) -> Net-(D7-Pad2)
- J7 pad 3: Net-(J6-Pad3) -> Net-(J7-Pad3)
- J7 pad 4: Net-(J6-Pad4) -> Net-(J7-Pad4)
Routing:
- net /3.3V_BBB: track 120.7 -> 249.5 mm, vias 0 -> 2
- net +24V: track 183.6 -> 300.5 mm
- net (no net): track 105.1 -> 0.00 mm, vias 1 -> 0
- net Net-(D5-Pad2): track 78.3 -> 170.5 mm
- net VCC: track 221.2 -> 168.5 mm
- net Net-(D10-Pad2): track 57.7 -> 105.3 mm
- net Net-(J7-Pad3): track 2.91 -> 50.0 mm
- net Net-(D12-Pad2): track 28.6 -> 74.8 mm
- net /AIn_BBB: track 85.7 -> 131.4 mm
- net Net-(J6-Pad4): track 141.9 -> 98.3 mm
- net Net-(D6-Pad2): track 53.3 -> 92.7 mm
- net Net-(J2-Pad2): track 0.00 -> 37.2 mm
- net Net-(J6-Pad3): track 66.4 -> 96.6 mm
- net Net-(J2-Pad1): track 0.00 -> 28.7 mm
- net Net-(J7-Pad4): track 77.4 -> 49.0 mm
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
Commit message: new hardware version
Parts:
- J2: footprint Connectors:USB_Micro-B -> Pin_Headers:Pin_Header_Straight_2x06_Pitch2.54mm
- moved R1 11.9 mm to (132.4, 117.1)
- moved J2 10.4 mm to (72.5, 74.4), turned to 270 degrees
- moved R2 8.05 mm to (164.2, 110.0), turned to 270 degrees
- moved R16 4.99 mm to (155.5, 124.4)
- moved R12 4.60 mm to (155.6, 118.8)
- moved D1 3.11 mm to (140.1, 121.7)
- moved K2 3.11 mm to (144.0, 121.7)
- moved R23 3.11 mm to (157.4, 109.5)
- moved R30 3.11 mm to (157.4, 104.2)
- moved D5 3.11 mm to (150.4, 114.4)
- moved D9 3.11 mm to (150.3, 106.5)
- moved J1 2.67 mm to (126.6, 132.0)
- moved Q1 1.48 mm to (138.8, 117.4), turned to 180 degrees
Connections:
- Beagle1 pad C1: Net-(Beagle1-PadC1) -> GND
- Beagle1 pad C2: Net-(Beagle1-PadC2) -> GND
- Beagle1 pad C43: Net-(Beagle1-PadC43) -> GND
- Beagle1 pad C44: Net-(Beagle1-PadC44) -> GND
- Beagle1 pad C45: Net-(Beagle1-PadC45) -> GND
- Beagle1 pad C46: Net-(Beagle1-PadC46) -> GND
Routing:
- net Net-(D5-Pad2): track 170.5 -> 99.6 mm
- net +24V: track 300.5 -> 242.9 mm, vias 0 -> 1
- net VCC: track 168.5 -> 199.5 mm
- net GND: track 74.4 -> 56.2 mm, vias 4 -> 6
- net /BBB_p1: track 39.0 -> 52.6 mm
- net Net-(D10-Pad2): track 105.3 -> 115.7 mm
- net Net-(J2-Pad1): track 28.7 -> 38.4 mm
- net Net-(J5-Pad3): track 91.0 -> 100.0 mm
- net Net-(J2-Pad3): track 24.1 -> 31.8 mm
- net Net-(J2-Pad2): track 37.2 -> 30.1 mm
- net Net-(D12-Pad2): track 74.8 -> 81.9 mm
- net /BBB_p3: track 9.71 -> 16.3 mm
- net Net-(D11-Pad2): track 39.4 -> 45.2 mm
- net /3.3V_BBB: track 249.5 -> 253.4 mm
- net Net-(D8-Pad1): track 14.3 -> 10.5 mm
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
Commit message: new hardware version
Parts:
- moved R20 8.00 mm to (174.3, 53.6), turned to 180 degrees
- moved R18 6.91 mm to (148.6, 53.2), turned to 180 degrees
- moved R24 6.46 mm to (180.4, 55.9)
- moved R21 6.17 mm to (154.5, 55.9)
- moved R10 5.71 mm to (150.3, 71.5), turned to 180 degrees
- moved R14 5.58 mm to (150.3, 76.6), turned to 180 degrees
- moved D6 2.49 mm to (150.1, 66.4)
- moved J1 2.04 mm to (126.5, 134.0)
- moved D8 1.96 mm to (175.3, 66.8)
- moved D12 1.50 mm to (174.4, 58.1)
- moved R8 1.02 mm to (188.6, 57.7)
- moved D10 0.77 mm to (148.6, 58.4)
Routing:
- net GND: track 56.2 -> 41.8 mm, vias 6 -> 4
- net Net-(D6-Pad2): track 96.2 -> 84.9 mm
- net Net-(D10-Pad2): track 115.7 -> 105.6 mm
- net Net-(D12-Pad2): track 81.9 -> 72.0 mm
- net VCC: track 199.5 -> 208.5 mm
- net Net-(J5-Pad3): track 100.0 -> 91.2 mm
- net Net-(J5-Pad4): track 93.7 -> 87.4 mm
- net +24V: track 242.9 -> 237.4 mm
- net Net-(D11-Pad2): track 45.2 -> 48.8 mm
- net /AIn_BBB: track 131.2 -> 134.6 mm
- net Net-(J6-Pad4): track 98.3 -> 100.4 mm
- net Net-(D5-Pad2): track 99.6 -> 101.4 mm
- net /BBB_p3: track 16.3 -> 17.7 mm
- net Net-(D12-Pad1): track 10.2 -> 8.93 mm
- net Net-(D11-Pad1): track 12.2 -> 10.9 mm
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