File: hardware/kicad/VBC.kicad_pcb (KiCad board)
At the start: 2 copper layers, 160 x 100.1 mm, 57 parts, among them J1 Conn_01x01, J10 Conn_01x01, J2 USB_OTG, J3 RJ25, J4 Conn_01x02, J5 RJ11, J6 RJ11, J7 RJ11, J8 RJ11, J9 USB_A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

Commit message: new hardware version
Parts:
- removed P1: CONN_01X01, Controle:LNLS_LOGO
- J9: moved to F.Cu
- moved J2 19.3 mm to (66.0, 92.6), turned to 180 degrees
- turned J9 to 270 degrees
Routing:
- net Net-(J2-Pad1): track 38.4 -> 16.9 mm
- net Net-(J2-Pad3): track 31.8 -> 43.0 mm
- net Net-(J2-Pad2): track 30.1 -> 21.9 mm

Commit message: new hardware version
Parts:
- added P1: CONN_01X01, Controle:LNLS_LOGO, F.Cu at (136.9, 148.3)
- Beagle1: moved to F.Cu
- moved Q2 2.23 mm to (169.5, 118.2)
- moved D5 1.80 mm to (150.3, 116.2)
- moved R23 0.42 mm to (157.5, 109.1)
Connections:
- Beagle1 pad B16: Net-(Beagle1-PadB16) -> /BBB_p3
- Beagle1 pad B18: Net-(Beagle1-PadB18) -> /BBB_p1
- Beagle1 pad C21: /BBB_p3 -> Net-(Beagle1-PadC21)
- Beagle1 pad C23: /BBB_p1 -> Net-(Beagle1-PadC23)
- J5 pad 2: Net-(D5-Pad2) -> GND
- J5 pad 4: Net-(J5-Pad4) -> GND
- J6 pad 2: Net-(D6-Pad2) -> GND
- J6 pad 4: Net-(J6-Pad4) -> GND
- J7 pad 2: Net-(D7-Pad2) -> GND
- J7 pad 4: Net-(J7-Pad4) -> GND
- J8 pad 2: Net-(D8-Pad2) -> GND
- J8 pad 4: Net-(J8-Pad4) -> GND
- K1 pad 11: Net-(J6-Pad4) -> Net-(K1-Pad11)
- K2 pad 11: Net-(J5-Pad4) -> Net-(K2-Pad11)
- K3 pad 11: Net-(J7-Pad4) -> Net-(K3-Pad11)
- K4 pad 11: Net-(J8-Pad4) -> Net-(K4-Pad11)
Routing:
- net Net-(J6-Pad4): track 100.4 -> 0.00 mm
- net /AIn_BBB: track 134.6 -> 35.1 mm
- net Net-(Beagle1-PadB35): track 0.00 -> 99.5 mm
- net Net-(J6-Pad3): track 96.3 -> 0.06 mm
- net Net-(D5-Pad2): track 101.4 -> 9.19 mm
- net Net-(J5-Pad4): track 87.4 -> 0.00 mm
- net Net-(D10-Pad2): track 105.6 -> 21.8 mm
- net Net-(D6-Pad2): track 84.9 -> 8.26 mm
- net VCC: track 208.5 -> 140.8 mm
- net Net-(D12-Pad2): track 72.0 -> 4.72 mm
- net Net-(J8-Pad3): track 63.9 -> 0.00 mm
- net Net-(J8-Pad4): track 62.7 -> 0.00 mm
- net Net-(D7-Pad2): track 65.3 -> 7.18 mm
- net /3.3V_BBB: track 253.8 -> 196.0 mm
- net Net-(J7-Pad4): track 49.0 -> 0.00 mm
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
Commit message: new hardware version
Parts:
- moved R20 10.8 mm to (184.2, 58.0), turned to 0 degrees
- moved R18 9.51 mm to (154.4, 60.8), turned to 0 degrees
- moved R7 2.09 mm to (194.9, 54.1), turned to 0 degrees
- moved R8 1.96 mm to (190.5, 58.3)
- moved R24 1.29 mm to (179.2, 55.3), turned to 180 degrees
- moved R21 0.36 mm to (154.2, 55.7)
Connections:
- Beagle1 pad B7: /BBB_p5 -> Net-(Beagle1-PadB7)
- Beagle1 pad B9: /BBB_p6 -> Net-(Beagle1-PadB9)
- Beagle1 pad C14: Net-(Beagle1-PadC14) -> /BBB_p5
- Beagle1 pad C16: Net-(Beagle1-PadC16) -> /BBB_p6
- J1 pad 1: Net-(J1-Pad1) -> GND
- J1 pad 2: (no net) -> GND
Routing:
- net VCC: track 140.8 -> 288.6 mm
- net Net-(J6-Pad3): track 0.06 -> 115.6 mm
- net Net-(Beagle1-PadB35): track 99.5 -> 0.00 mm
- net /3.3V_BBB: track 196.0 -> 102.5 mm
- net Net-(D10-Pad2): track 21.8 -> 97.6 mm
- net /BBB_p4: track 1.45 -> 72.1 mm
- net Net-(J8-Pad3): track 0.00 -> 66.1 mm
- net Net-(D12-Pad2): track 4.72 -> 58.4 mm
- net /BBB_p2: track 14.1 -> 58.7 mm
- net /AIn_BBB: track 35.1 -> 59.4 mm
- net Net-(Beagle1-PadB11): track 19.8 -> 0.00 mm
- net Net-(Beagle1-PadB23): track 17.8 -> 0.00 mm
- net /BBB_p5: track 15.0 -> 26.8 mm
- net +24V: track 237.4 -> 245.2 mm
- net /BBB_p6: track 45.5 -> 53.0 mm
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
Commit message: new hardware version
Routing:
- net GND: track 5.29 -> 108.0 mm, vias 4 -> 5
- net Net-(J1-Pad1): track 0.57 -> 0.00 mm

Commit message: new hardware version
Parts:
- moved P1 104.8 mm to (101.5, 49.6)
Routing:
- net GND: track 108.0 -> 84.0 mm
- net +24V: track 245.2 -> 240.0 mm, vias 1 -> 2
- net /3.3V_BBB: track 102.5 -> 105.9 mm
- net Net-(J8-Pad3): track 66.1 -> 67.9 mm
- net Net-(D12-Pad2): track 58.4 -> 59.8 mm

Commit message: minor changes in hardware files
Connections:
- J1 pad 1: GND -> Net-(J1-Pad1)
- J1 pad 2: GND -> (no net)
- J5 pad 1: Net-(D9-Pad2) -> GND
- J5 pad 2: GND -> Net-(J5-Pad2)
- J5 pad 3: Net-(J5-Pad3) -> GND
- J5 pad 4: GND -> Net-(D9-Pad2)
- J6 pad 1: Net-(D10-Pad2) -> GND
- J6 pad 2: GND -> Net-(J6-Pad2)
- J6 pad 3: Net-(J6-Pad3) -> GND
- J6 pad 4: GND -> Net-(D10-Pad2)
- J7 pad 1: Net-(D11-Pad2) -> GND
- J7 pad 2: GND -> Net-(J7-Pad2)
- J7 pad 3: Net-(J7-Pad3) -> GND
- J7 pad 4: GND -> Net-(D11-Pad2)
- J8 pad 1: Net-(D12-Pad2) -> GND
- J8 pad 2: GND -> Net-(J8-Pad2)
- J8 pad 3: Net-(J8-Pad3) -> GND
- J8 pad 4: GND -> Net-(D12-Pad2)
- K1 pad 9: Net-(J6-Pad3) -> Net-(J6-Pad2)
- K2 pad 9: Net-(J5-Pad3) -> Net-(J5-Pad2)
- K3 pad 9: Net-(J7-Pad3) -> Net-(J7-Pad2)
- K4 pad 9: Net-(J8-Pad3) -> Net-(J8-Pad2)
Routing:
- net Net-(J6-Pad3): track 115.6 -> 0.00 mm
- net Net-(J6-Pad2): track 0.00 -> 115.6 mm
- net Net-(J5-Pad3): track 89.4 -> 0.00 mm
- net Net-(J5-Pad2): track 0.00 -> 89.4 mm
- net Net-(J8-Pad3): track 67.9 -> 0.00 mm
- net Net-(J8-Pad2): track 0.00 -> 67.9 mm
- net Net-(J7-Pad3): track 59.9 -> 0.00 mm
- net Net-(J7-Pad2): track 0.00 -> 59.9 mm
- net Net-(J1-Pad1): track 0.00 -> 0.57 mm
- net GND: track 84.0 -> 83.5 mm
