File: hardware/kicad/_autosave-VBC.kicad_pcb (KiCad board)
At the start: 2 copper layers, 160 x 100.1 mm, 57 parts, among them J1 Conn_01x01, J10 Conn_01x01, J2 USB_OTG, J3 RJ25, J4 Conn_01x02, J5 RJ11, J6 RJ11, J7 RJ11, J8 RJ11, J9 USB_A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

Commit message: new hardware version
Parts:
- moved R20 10.8 mm to (184.2, 58.0), turned to 0 degrees
- moved R18 9.51 mm to (154.4, 60.8), turned to 0 degrees
- moved Q2 2.23 mm to (169.5, 118.2)
- moved R7 2.09 mm to (194.9, 54.1), turned to 0 degrees
- moved R8 1.96 mm to (190.5, 58.3)
- moved D5 1.80 mm to (150.3, 116.2)
- moved R24 1.29 mm to (179.2, 55.3), turned to 180 degrees
- moved R23 0.42 mm to (157.5, 109.1)
- moved R21 0.36 mm to (154.2, 55.7)
Connections:
- Beagle1 pad B7: /BBB_p5 -> Net-(Beagle1-PadB7)
- Beagle1 pad B9: /BBB_p6 -> Net-(Beagle1-PadB9)
- Beagle1 pad C14: Net-(Beagle1-PadC14) -> /BBB_p5
- Beagle1 pad C16: Net-(Beagle1-PadC16) -> /BBB_p6
- J5 pad 2: Net-(D5-Pad2) -> GND
- J5 pad 4: Net-(J5-Pad4) -> GND
- J6 pad 2: Net-(J6-Pad2) -> GND
- J6 pad 4: Net-(J6-Pad2) -> GND
- J7 pad 2: Net-(D7-Pad2) -> GND
- J7 pad 4: Net-(J7-Pad4) -> GND
- J8 pad 2: Net-(D8-Pad2) -> GND
- J8 pad 4: Net-(J8-Pad4) -> GND
- K2 pad 11: Net-(J5-Pad4) -> Net-(K2-Pad11)
- K3 pad 11: Net-(J7-Pad4) -> Net-(K3-Pad11)
- K4 pad 11: Net-(J8-Pad4) -> Net-(K4-Pad11)
Routing:
- net VCC: track 140.8 -> 288.6 mm
- net Net-(J6-Pad3): track 0.06 -> 115.6 mm
- net Net-(Beagle1-PadB35): track 99.5 -> 0.00 mm
- net /3.3V_BBB: track 196.0 -> 102.5 mm
- net Net-(J5-Pad3): track 0.74 -> 89.4 mm
- net Net-(D10-Pad2): track 21.8 -> 97.6 mm
- net Net-(D9-Pad2): track 5.99 -> 80.5 mm
- net /BBB_p4: track 1.45 -> 72.1 mm
- net Net-(J8-Pad3): track 0.00 -> 66.1 mm
- net Net-(J7-Pad3): track 0.00 -> 59.9 mm
- net Net-(D12-Pad2): track 4.72 -> 58.4 mm
- net /BBB_p2: track 14.1 -> 58.7 mm
- net Net-(D11-Pad2): track 5.70 -> 38.9 mm
- net /AIn_BBB: track 35.1 -> 59.4 mm
- net GND: track 26.7 -> 5.29 mm, vias 3 -> 4
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