File: hardware/kicad/VBC.sch (KiCad schematic (older format))
At the start: 36 parts, among them J1 Conn_01x01, J10 Conn_01x01, J2 USB_OTG, J3 RJ25, J4 Conn_01x02, J5 RJ11, J6 RJ11, J7 RJ11, J8 RJ11, J9 USB_A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

Commit message: added relay LED status in schematic
Parts:
- removed U2: TS5A21366, Controle:VSSOP-8, symbol TS5A21366
- added D10, D11, D12, D9: LED red, LEDs:LED_0805, symbol LED
- added D5, D6, D7, D8: LED green, LEDs:LED_0805, symbol LED
- added R10, R11, R17, R19, R21, R24, R26, R28: 2k2, Resistors_SMD:R_0805, symbol R
- added R12, R13, R14, R15, R30, R31, R32, R33: 180R, Resistors_SMD:R_0805, symbol R
- added R16, R18, R20, R22, R23, R25, R27, R29: 10k, Resistors_SMD:R_0805, symbol R
- J2: symbol USB_OTG -> USB_OTG-RESCUE-VBC
- J9: symbol USB_A -> USB_A-RESCUE-VBC
Connections:
- net labels removed: K1_P11, K1_P6, K1_P8, K1_P9, K2_P11, K2_P6, K2_P8, K2_P9, K3_P11, K3_P6, K3_P8, K3_P9, K4_P11, K4_P6, K4_P8, K4_P9
- wire segments 65 -> 158
- no-connect marks 101 -> 92
Other:
- moved on the sheet: J5

Commit message: new hardware version
Parts:
- removed R25, R27, R29: 10k, Resistors_SMD:R_0805, symbol R
- removed R26, R28: 2k2, Resistors_SMD:R_0805, symbol R
- removed R31, R32, R33: 180R, Resistors_SMD:R_0805, symbol R
- removed R9: 330K, Resistors_SMD:R_0805, symbol R
- removed U3: LT3080, TO_SOT_Packages_SMD:SOT-223, symbol LT3080
- D10, D11, D12, D5, D6, D7, D8, D9: footprint LEDs:LED_0805 -> LEDs:LED_0805_HandSoldering
- Q4: footprint TO_SOT_Packages_SMD:SOT-23 -> Resistors_SMD:R_0805_HandSoldering
- R1, R2, R3, R4, R5, R6, R7, R8: footprint Resistors_SMD:R_0805 -> Resistors_SMD:R_0805_HandSoldering
- R10, R11, R17, R19, R21, R24: value 2k2 -> 4k7; footprint Resistors_SMD:R_0805 -> Resistors_SMD:R_0805_HandSoldering
- R12, R13, R14, R15: value 180R -> 4k7; footprint Resistors_SMD:R_0805 -> Resistors_SMD:R_0805_HandSoldering
- R16, R18, R20, R22, R23: value 10k -> 4k7; footprint Resistors_SMD:R_0805 -> Resistors_SMD:R_0805_HandSoldering
- R30: value 180R -> 4k7
Connections:
- net VAT_P1 is gone; now on net 3.3V_BBB: J3.1
- net VAT_P6 is gone; now on net 3.3V_BBB: J3.6
- net GND: now also R10.2, R11.2, R17.2, R19.2, R21.2, R24.2
- net 3.3V_BBB: now reaches Beagle1.C3
- net at J6.2, K1.6 (R1): now also D6.2 (A); no longer R17.1
- net at J6.1, K1.8 (T1): now also D10.2 (A); no longer R24.1
- net at J5.2, K2.6 (R1): now also D5.2 (A); no longer R10.1
- net at J5.1, K2.8 (T1): now also D9.2 (A); no longer R11.1
- net at J8.2, K4.6 (R1): now also D8.2 (A); no longer R21.1
- net at J8.1, K4.8 (T1): now also D12.2 (A)
- net at J7.2, K3.6 (R1): now also D7.2 (A); no longer R19.1
- net at J7.1, K3.8 (T1): now also D11.2 (A)
- net at D9.1 (K), R30.1: now also R23.1
- net at D5.1 (K), R12.1: now also R16.1
- net at D12.1 (K): now also R20.1, R24.1
- net at D8.1 (K): now also R13.1, R17.1; no longer R15.1
- net at D10.1 (K): now also R18.1, R21.1
- net at D6.1 (K): now also R10.1, R14.1; no longer R13.1
- net at D11.1 (K): now also R19.1, R22.1
- net at D7.1 (K): now also R11.1, R15.1; no longer R14.1
- no-connect marks 92 -> 91
Other:
- moved on the sheet: D5, D9, R12, R23, R30

Commit message: new hardware version
Connections:
- net 3.3V_BBB: now also Beagle1.C4; no longer Beagle1.C3
- net GND: now also Beagle1.C1, Beagle1.C2, Beagle1.C43, Beagle1.C44, Beagle1.C45, Beagle1.C46
- no-connect marks 91 -> 86
Changed lines of the file:
@@
 NoConn ~ 10110 2880
 NoConn ~ 10110 3180
-NoConn ~ 10110 2580
-NoConn ~ 10610 2680
-NoConn ~ 10610 2580
 NoConn ~ 10610 2880
 NoConn ~ 10610 2980
@@
 NoConn ~ 10610 4480
 NoConn ~ 10610 4580
-NoConn ~ 10610 4680
-NoConn ~ 10110 4680
 NoConn ~ 10110 4580
 NoConn ~ 10110 4480
@@
 $EndComp
 NoConn ~ 9450 4785
-NoConn ~ 10110 4780
-NoConn ~ 10610 4780
 $Comp
 L GND #PWR023
@@
 Text Label 5925 2720 2    60   ~ 0
 3.3V_BBB
-Text Label 10110 2680 2    60   ~ 0
+Text Label 10610 2680 0    60   ~ 0
 3.3V_BBB
 $Comp
@@
 	-1   0    0    1
 $EndComp
+NoConn ~ 10110 2680
+NoConn ~ 2900 6985
+$Comp
+L GND #PWR?
+U 1 1 5B3BC7A9
+P 10110 2580
+F 0 "#PWR?" H 10110 2330 50  0001 C CNN
+F 1 "GND" H 10110 2430 50  0000 C CNN
+F 2 "" H 10110 2580 50  0001 C CNN
+F 3 "" H 10110 2580 50  0001 C CNN
+	1    10110 2580
+	0    1    1    0
+$EndComp
+$Comp
+L GND #PWR?
+U 1 1 5B3BC8DF
+P 10610 2580
+F 0 "#PWR?" H 10610 2330 50  0001 C CNN
+F 1 "GND" H 10610 2430 50  0000 C CNN
+F 2 "" H 10610 2580 50  0001 C CNN
+F 3 "" H 10610 2580 50  0001 C CNN
+	1    10610 2580
+	0    -1   -1   0
+$EndComp
+$Comp
+L GND #PWR?
+U 1 1 5B3BCBAB
+P 10110 4780
+F 0 "#PWR?" H 10110 4530 50  0001 C CNN
+F 1 "GND" H 10110 4630 50  0000 C CNN
+F 2 "" H 10110 4780 50  0001 C CNN
+F 3 "" H 10110 4780 50  0001 C CNN
+	1    10110 4780
+	1    0    0    -1
+$EndComp
+$Comp
+L GND #PWR?
+U 1 1 5B3BCF5F
+P 10610 4780
+F 0 "#PWR?" H 10610 4530 50  0001 C CNN
+F 1 "GND" H 10610 4630 50  0000 C CNN
+F 2 "" H 10610 4780 50  0001 C CNN
+F 3 "" H 10610 4780 50  0001 C CNN
+	1    10610 4780
+	1    0    0    -1
+$EndComp
+Wire Wire Line
+	10610 4680 10610 4780
+Wire Wire Line
+	10110 4680 10110 4780
 $EndSCHEMATC

Commit message: new hardware version
Connections:
- net BBB_p1: now also Beagle1.B18; no longer Beagle1.C23
- net BBB_p3: now also Beagle1.B16; no longer Beagle1.C21
- net BBB_p5: now also Beagle1.C14; no longer Beagle1.B7
- net BBB_p6: now also Beagle1.C16; no longer Beagle1.B9
- net GND: now also J5.2, J5.4, J6.2, J6.4, J7.2, J7.4, J8.2, J8.4
- net at K1.11 (R2): no longer J6.4
- net at D6.2 (A), K1.6 (R1): no longer J6.2
- net at K2.11 (R2): no longer J5.4
- net at D5.2 (A), K2.6 (R1): no longer J5.2
- net at K4.11 (R2): no longer J8.4
- net at D8.2 (A), K4.6 (R1): no longer J8.2
- net at K3.11 (R2): no longer J7.4
- net at D7.2 (A), K3.6 (R1): no longer J7.2
- no-connect marks 86 -> 89
Changed lines of the file:
@@
 Text Label 6300 1530 3    60   ~ 0
 VAT_P6
-Text Label 10110 3680 2    60   ~ 0
+Text Label 9450 3385 0    60   ~ 0
 BBB_p1
 Text Label 10610 3680 0    60   ~ 0
 BBB_p2
-Text Label 10110 3580 2    60   ~ 0
+Text Label 9450 3285 0    60   ~ 0
 BBB_p3
 Text Label 10610 3080 0    60   ~ 0
@@
 	1    0    0    -1
 $EndComp
-Text Label 8950 2985 2    60   ~ 0
+Text Label 10610 3280 0    60   ~ 0
 BBB_p6
-Text Label 8950 2885 2    60   ~ 0
+Text Label 10610 3180 0    60   ~ 0
 BBB_p5
 NoConn ~ 9715 1445
@@
 NoConn ~ 9450 3085
 NoConn ~ 9450 3185
-NoConn ~ 9450 3285
 NoConn ~ 8950 3285
 NoConn ~ 8950 3185
@@
 NoConn ~ 10110 2880
 NoConn ~ 10110 3180
-NoConn ~ 10610 2880
-NoConn ~ 10610 2980
-NoConn ~ 10610 3180
-NoConn ~ 10610 3280
 NoConn ~ 10610 3380
 NoConn ~ 10610 3480
@@
 NoConn ~ 10110 3480
 NoConn ~ 10110 3380
-NoConn ~ 9450 3385
 NoConn ~ 9450 3485
 NoConn ~ 9450 3585
@@
 Connection ~ 3090 6490
 Connection ~ 3055 2760
-Connection ~ 2835 915
 Connection ~ 2835 1865
 Wire Wire Line
@@
 	3230 6390 3090 6390
 Wire Wire Line
-	3090 6090 3230 6090
-Wire Wire Line
-	3090 5990 3090 6090
+	2960 6090 3230 6090
 Wire Wire Line
 	2540 6190 3230 6190
 Wire Wire Line
-	3230 6290 2540 6290
-Wire Wire Line
-	2540 5990 3090 5990
-Wire Wire Line
 	2530 4565 3085 4565
 Wire Wire Line
@@
 	3220 4465 3080 4465
 Wire Wire Line
-	3080 4165 3220 4165
-Wire Wire Line
-	3080 4065 3080 4165
+	2920 4165 3220 4165
 Wire Wire Line
 	2530 4265 3220 4265
 Wire Wire Line
-	3220 4365 2530 4365
-Wire Wire Line
-	2530 4065 3080 4065
-Wire Wire Line
 	3055 2760 2505 2760
 Wire Wire Line
@@
 	3195 2660 3055 2660
 Wire Wire Line
-	3055 2360 3195 2360
-Wire Wire Line
-	3055 2260 3055 2360
-Wire Wire Line
 	2505 2460 3195 2460
 Wire Wire Line
-	3195 2560 2505 2560
-Wire Wire Line
-	2505 2260 3055 2260
-Wire Wire Line
 	2450 1115 3100 1115
 Wire Wire Line
 	3140 1015 3000 1015
 Wire Wire Line
-	3000 715  3140 715
-Wire Wire Line
-	3000 615  3000 715
-Wire Wire Line
 	2450 815  3140 815
-Wire Wire Line
-	3140 915  2450 915
-Wire Wire Line
-	2450 615  3000 615
 Wire Wire Line
 	1705 3645 1705 3755
@@
 	3100 1545 3320 1545
 Wire Wire Line
-	3100 1865 3320 1865
+	2965 1865 3320 1865
 Wire Wire Line
 	3320 1865 3320 1845
@@
 	3055 3295 3275 3295
 Wire Wire Line
-	3055 3615 3275 3615
+	2920 3615 3275 3615
 Wire Wire Line
 	3275 3615 3275 3595
@@
 	3085 5035 3305 5035
 Wire Wire Line
-	3085 5355 3305 5355
+	2960 5355 3305 5355
 Wire Wire Line
 	3305 5355 3305 5335
 Wire Wire Line
 	2825 6655 2825 6290
-Connection ~ 2825 6290
 Wire Wire Line
 	3085 4565 3085 4670
@@
 Wire Wire Line
 	2820 4670 2820 4365
-Connection ~ 2820 4365
 Wire Wire Line
 	3100 1115 3100 1180
 Wire Wire Line
-	2835 1180 2835 915
-Wire Wire Line
-	2790 2930 2790 2560
-Connection ~ 2790 2560
+	2835 915  2835 1180
 Wire Wire Line
 	6150 2405 6135 2405
@@
 NoConn ~ 2900 6985
 $Comp
-L GND #PWR?
+L GND #PWR032
 U 1 1 5B3BC7A9
 P 10110 2580
-F 0 "#PWR?" H 10110 2330 50  0001 C CNN
+F 0 "#PWR032" H 10110 2330 50  0001 C CNN
 F 1 "GND" H 10110 2430 50  0000 C CNN
 F 2 "" H 10110 2580 50  0001 C CNN
@@
 $EndComp
 $Comp
-L GND #PWR?
+L GND #PWR033
 U 1 1 5B3BC8DF
 P 10610 2580
-F 0 "#PWR?" H 10610 2330 50  0001 C CNN
+F 0 "#PWR033" H 10610 2330 50  0001 C CNN
 F 1 "GND" H 10610 2430 50  0000 C CNN
 F 2 "" H 10610 2580 50  0001 C CNN
@@
 $EndComp
 $Comp
-L GND #PWR?
+L GND #PWR034
 U 1 1 5B3BCBAB
 P 10110 4780
-F 0 "#PWR?" H 10110 4530 50  0001 C CNN
+F 0 "#PWR034" H 10110 4530 50  0001 C CNN
 F 1 "GND" H 10110 4630 50  0000 C CNN
 F 2 "" H 10110 4780 50  0001 C CNN
@@
 $EndComp
 $Comp
-L GND #PWR?
+L GND #PWR035
 U 1 1 5B3BCF5F
 P 10610 4780
-F 0 "#PWR?" H 10610 4530 50  0001 C CNN
+F 0 "#PWR035" H 10610 4530 50  0001 C CNN
 F 1 "GND" H 10610 4630 50  0000 C CNN
 F 2 "" H 10610 4780 50  0001 C CNN
@@
 Wire Wire Line
 	10110 4680 10110 4780
+Wire Wire Line
+	2790 2560 2505 2560
+Wire Wire Line
+	3195 2560 3110 2560
+Wire Wire Line
+	3110 2560 3110 2360
+Wire Wire Line
+	2965 2360 3195 2360
+NoConn ~ 2505 2260
+Wire Wire Line
+	2790 2560 2790 2930
+Wire Wire Line
+	2835 915  2450 915
+Wire Wire Line
+	2965 2360 2965 1865
+Connection ~ 3110 2360
+Wire Wire Line
+	2965 915  2965 1870
+Connection ~ 2965 1870
+Wire Wire Line
+	3140 715  3140 915
+Wire Wire Line
+	3140 915  2965 915
+Wire Wire Line
+	2820 4365 2530 4365
+Wire Wire Line
+	3080 4165 3080 4365
+Wire Wire Line
+	3080 4365 3220 4365
+Wire Wire Line
+	2920 4165 2920 3615
+Connection ~ 3080 4165
+Wire Wire Line
+	2825 6290 2540 6290
+Wire Wire Line
+	3230 6290 3090 6290
+Wire Wire Line
+	3090 6290 3090 6090
+Wire Wire Line
+	2960 6090 2960 5355
+Connection ~ 3090 6090
+NoConn ~ 2540 5990
+NoConn ~ 2530 4065
+NoConn ~ 2450 615
+NoConn ~ 15530 2965
+NoConn ~ 10610 2880
+NoConn ~ 10610 2980
+NoConn ~ 8950 2885
+NoConn ~ 8950 2985
 $EndSCHEMATC

Commit message: new hardware version
Connections:
- no-connect marks 89 -> 90
Changed lines of the file:
@@
 NoConn ~ 8950 2885
 NoConn ~ 8950 2985
+NoConn ~ 10165 1610
 $EndSCHEMATC

Commit message: minor changes in hardware files
Parts:
- D10, D11, D12, D5, D6, D7, D8, D9: symbol LED -> LED-RESCUE-VBC
Connections:
- net GND: now also J5.1, J5.3, J6.1, J6.3, J7.1, J7.3, J8.1, J8.3; no longer J5.2, J5.4, J6.2, J6.4, J7.2, J7.4, J8.2, J8.4
- net at D10.2 (A), K1.8 (T1): now also J6.4; no longer J6.1
- net at K1.9 (T2): now also J6.2; no longer J6.3
- net at D9.2 (A), K2.8 (T1): now also J5.4; no longer J5.1
- net at K2.9 (T2): now also J5.2; no longer J5.3
- net at D12.2 (A), K4.8 (T1): now also J8.4; no longer J8.1
- net at K4.9 (T2): now also J8.2; no longer J8.3
- net at D11.2 (A), K3.8 (T1): now also J7.4; no longer J7.1
- net at K3.9 (T2): now also J7.2; no longer J7.3
Changed lines of the file:
@@
 F 3 "" H 3740 865 60  0000 C CNN
 	1    3740 865
-	0    1    -1   0
+	0    1    1    0
 $EndComp
 $Comp
@@
 F 3 "" H 3795 2510 60  0000 C CNN
 	1    3795 2510
-	0    1    -1   0
+	0    1    1    0
 $EndComp
 $Comp
@@
 F 3 "" H 3820 4315 60  0000 C CNN
 	1    3820 4315
-	0    1    -1   0
+	0    1    1    0
 $EndComp
 $Comp
@@
 F 3 "" H 3830 6240 60  0000 C CNN
 	1    3830 6240
-	0    1    -1   0
+	0    1    1    0
 $EndComp
 $Comp
@@
 $EndComp
 $Comp
-L LED D9
+L LED-RESCUE-VBC D9
 U 1 1 5B3AAF77
 P 3100 1330
@@
 $EndComp
 $Comp
-L LED D5
+L LED-RESCUE-VBC D5
 U 1 1 5B3AE242
 P 2835 1330
@@
 $EndComp
 $Comp
-L LED D12
+L LED-RESCUE-VBC D12
 U 1 1 5B3AD5EA
 P 3090 6805
@@
 $EndComp
 $Comp
-L LED D8
+L LED-RESCUE-VBC D8
 U 1 1 5B3AD602
 P 2825 6805
@@
 $EndComp
 $Comp
-L LED D10
+L LED-RESCUE-VBC D10
 U 1 1 5B3AEC39
 P 3055 3080
@@
 $EndComp
 $Comp
-L LED D6
+L LED-RESCUE-VBC D6
 U 1 1 5B3AEC51
 P 2790 3080
@@
 $EndComp
 $Comp
-L LED D11
+L LED-RESCUE-VBC D11
 U 1 1 5B3AF3CE
 P 3085 4820
@@
 $EndComp
 $Comp
-L LED D7
+L LED-RESCUE-VBC D7
 U 1 1 5B3AF3E6
 P 2820 4820
