File: hardware/kicad/VBC v2.0/USB_converter_485.sch (KiCad schematic (older format))
At the start: 33 parts, among them P2 USB Mini-B, P3 RJ25, P4 RJ25, P5 CONN_01X01, P6 CONN_01X01, SW1 SW_DIP_2, U1 TS5A21366, U2 TS5A21366, U3 FT232RL, U4 IL3685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

Commit message: new hardware version - v2.0
Parts:
- D13, D14: footprint Conversor USB-RS485:LED_SMD -> Controle:LED_para_painel_KINGBRIGHT
- P2: footprint Conversor USB-RS485:USB_Mini-B -> Controle:USB_Mini-B
- P3, P4: footprint Conversor USB-RS485:RJ25 -> Controle:RJ25_(conversor)
- U5: footprint Conversor USB-RS485:DCR010505U -> Controle:DCR01XXXXU
Changed lines of the file:
@@
 F 0 "D13" V 1785 4235 50  0000 R CNN
 F 1 "LED" V 1685 4235 50  0001 R CNN
-F 2 "Conversor USB-RS485:LED_SMD" V 1735 4335 50  0001 C CNN
+F 2 "Controle:LED_para_painel_KINGBRIGHT" V 1735 4335 50  0001 C CNN
 F 3 "" V 1735 4335 50  0000 C CNN
 	1    1735 4335
@@
 F 0 "D14" V 2585 4235 50  0000 R CNN
 F 1 "LED" V 2485 4235 50  0001 R CNN
-F 2 "Conversor USB-RS485:LED_SMD" V 2535 4335 50  0001 C CNN
+F 2 "Controle:LED_para_painel_KINGBRIGHT" V 2535 4335 50  0001 C CNN
 F 3 "" V 2535 4335 50  0000 C CNN
 	1    2535 4335
@@
 F 0 "P3" H 5500 4750 50  0000 C CNN
 F 1 "RJ25" H 5500 3950 50  0001 C CNN
-F 2 "Conversor USB-RS485:RJ25" H 5500 4350 50  0001 C CNN
+F 2 "Controle:RJ25_(conversor)" H 5500 4350 50  0001 C CNN
 F 3 "" H 5500 4350 50  0000 C CNN
 	1    5500 4350
@@
 F 0 "U5" H 9305 3120 60  0000 L CNN
 F 1 "DCR010505U" H 9305 3020 60  0000 L CNN
-F 2 "Conversor USB-RS485:DCR010505U" H 9405 2470 60  0001 C CNN
+F 2 "Controle:DCR01XXXXU" H 9405 2470 60  0001 C CNN
 F 3 "" H 9405 2470 60  0000 C CNN
 	1    9755 2170
@@
 F 0 "P2" H 2585 1985 50  0000 L CNN
 F 1 "USB Mini-B" H 2585 1885 50  0000 L CNN
-F 2 "Conversor USB-RS485:USB_Mini-B" V 2785 1385 50  0001 C CNN
+F 2 "Controle:USB_Mini-B" V 2785 1385 50  0001 C CNN
 F 3 "" V 2785 1385 50  0000 C CNN
 	1    2835 1485
@@
 F 0 "P4" H 6650 7560 50  0000 C CNN
 F 1 "RJ25" H 6650 6760 50  0001 C CNN
-F 2 "Conversor USB-RS485:RJ25" H 6650 7160 50  0001 C CNN
+F 2 "Controle:RJ25_(conversor)" H 6650 7160 50  0001 C CNN
 F 3 "" H 6650 7160 50  0000 C CNN
 	1    6650 7160
