File: hardware/kicad/VBC v2.0/VBC_v2-0.kicad_pcb (KiCad board)
At the start: 2 copper layers, 160 x 100.1 mm, 88 parts, among them J1 Conn_01x01, J10 Conn_01x01, J3 RJ25, J4 Conn_01x02, J5 RJ11, J6 RJ11, J7 RJ11, J8 RJ11, K1 RELAY_Metaltex, K2 RELAY_Metaltex, K3 RELAY_Metaltex, K4 RELAY_Metaltex, P1 USB Mini-B, P3 RJ25, Q1 BC817, Q2 BC817, Q3 BC817, Q4 BC817, SW1 SW_DIP_2, U1 FT232RL, U2 IL3685, U3 DCR010505U, U4 TS5A21366, U5 TS5A21366

Commit message: new hardware version - v2.0
Parts:
- removed Fiducial: Fiducial_1mm_Dia_2.54mm_Outer_CopperTop, Fiducials:Fiducial_1mm_Dia_2.54mm_Outer_CopperTop
- removed Fiducial: Fiducial_1mm_Dia_2.54mm_Outer_CopperBottom, Fiducials:Fiducial_1mm_Dia_2.54mm_Outer_CopperBottom
- removed the G*** at (174.8, -49.6)
- added G***: LOGO, Controle:LNLS_LOGO_Silk, F.Cu at (252.8, 116.8)
- added P4: RJ25, Conversor USB-RS485:RJ25, F.Cu at (119.4, 104.1)
- added R34: 5k, Resistors_SMD:R_0805_HandSoldering, F.Cu at (256.2, 71.7)
- added R35: 10k, Resistors_SMD:R_0805_HandSoldering, F.Cu at (256.3, 65.8)
- J8: renamed from J10; moved to F.Cu
- R21: renamed from R6; value 5k -> 10k
- R22: renamed from R5; value 10k -> 5k
- moved R22 9.22 mm to (246.9, 71.3), turned to 270 degrees
- moved P3 7.00 mm to (119.4, 87.1)
- moved D13 5.00 mm to (117.8, 75.2)
- moved SW1 5.00 mm to (119.3, 116.4)
- moved R25 2.70 mm to (144.8, 103.4)
- moved R30 2.70 mm to (141.9, 103.4)
- moved U1 2.70 mm to (136.4, 103.7)
- moved C6 2.56 mm to (184.0, 107.1)
- moved REF** 2.46 mm to (116.6, 129.6)
- moved D14 2.00 mm to (117.8, 69.1)
- moved R21 1.36 mm to (251.1, 68.6)
- turned R23 to 0 degrees
- renumbered C7 to C11, C1 to C2, C2 to C3, C3 to C4, C4 to C5, C5 to C6, C8 to C7, C9 to C8, C6 to C9, D11 to D10, D12 to D11, D9 to D12, D1 to D13, D6 to D5, D7 to D6, D8 to D7, D5 to D8, D10 to D9, J5 to J1, J6 to J2, J7 to J3, J8 to J4, J3 to J5, J4 to J6, J1 to J7, K2 to K1, K1 to K2, P1 to P2, Q3 to Q2, Q2 to Q3, R11 to R10, R13 to R11, R21 to R13, R19 to R14, R24 to R15, R30 to R16, R18 to R17, R22 to R18, R20 to R19, R3 to R2, R23 to R20, R8 to R23, R7 to R24, R2 to R25, R1 to R26, R3 to R27, R4 to R28, R2 to R3, R8 to R30, R9 to R31, R6 to R32, R7 to R33, R10 to R5, R15 to R6, R17 to R7, R16 to R8, R14 to R9, U4 to U1, U5 to U2, U1 to U3, U2 to U4, U3 to U5
Connections:
- net /GND_ISOLATED renamed /USB_converter_485./GND_ISOLATED
- net /RS485+ renamed /USB_converter_485./RS485+
- net /RS485- renamed /USB_converter_485./RS485-
- net /RXD renamed /USB_converter_485./RXD
- net /RXLED# renamed /USB_converter_485./RXLED#
- net /TXD renamed /USB_converter_485./TXD
- net /TXDEN renamed /USB_converter_485./TXDEN
- net /TXLED# renamed /USB_converter_485./TXLED#
- net /USB_D+ renamed /USB_converter_485./USB_D+
- net /USB_D- renamed /USB_converter_485./USB_D-
- C10 pad 1: /5V_ISOLATED -> /USB_converter_485./5V_ISOLATED
- C11 pad 1: /5V_ISOLATED -> /USB_converter_485./5V_ISOLATED
- C9 pad 1: /5V_ISOLATED -> /USB_converter_485./5V_ISOLATED
- D13 pad 2: Net-(D1-Pad2) -> Net-(D13-Pad2)
- D14 pad 2: Net-(D2-Pad2) -> Net-(D14-Pad2)
- J7 pad 1: (no net) -> GND
- J7 pad 2: GND -> (no net)
- P3 pad 6: /5V_ISOLATED -> (no net)
- R21 pad 1: /AIn_BBB -> Net-(R21-Pad1)
- R21 pad 2: GND -> /AIn_BBB
- R22 pad 1: Net-(C1-Pad1) -> /AIn_BBB
- R22 pad 2: /AIn_BBB -> GND
- R26 pad 2: /5V_ISOLATED -> /USB_converter_485./5V_ISOLATED
- R28 pad 2: Net-(D1-Pad2) -> Net-(D13-Pad2)
- R29 pad 2: Net-(D2-Pad2) -> Net-(D14-Pad2)
- R33 pad 1: /5V_ISOLATED -> /USB_converter_485./5V_ISOLATED
- SW1 pad 1: /5V_ISOLATED -> /USB_converter_485./5V_ISOLATED
- SW1 pad 3: /5V_ISOLATED -> /USB_converter_485./5V_ISOLATED
- U1 pad 8: /5V_ISOLATED -> /USB_converter_485./5V_ISOLATED
- U2 pad 8: /5V_ISOLATED -> /USB_converter_485./5V_ISOLATED
- U4 pad 16: /5V_ISOLATED -> /USB_converter_485./5V_ISOLATED
- U5 pad 14: /5V_ISOLATED -> /USB_converter_485./5V_ISOLATED
Routing:
- net /5V_ISOLATED: track 151.4 -> 0.00 mm, vias 2 -> 0
- net GND: track 263.6 -> 409.2 mm
- net /USB_converter_485./5V_ISOLATED: track 0.00 -> 142.7 mm, vias 0 -> 2
- net /USB_converter_485./RS485+: track 70.4 -> 112.0 mm
- net Net-(D13-Pad2): track 0.00 -> 22.7 mm, vias 0 -> 1
- net Net-(D14-Pad2): track 0.00 -> 21.8 mm, vias 0 -> 1
- net Net-(D2-Pad2): track 27.5 -> 6.58 mm, vias 1 -> 0
- net Net-(D1-Pad2): track 28.5 -> 7.62 mm, vias 1 -> 0
- net /USB_converter_485./RS485-: track 55.4 -> 73.5 mm
- net /3.3V_BBB: track 105.9 -> 96.2 mm
- net /AIn_BBB: track 59.4 -> 50.1 mm
- net Net-(R30-Pad2): track 21.9 -> 29.1 mm
- net Net-(R34-Pad2): track 0.00 -> 7.09 mm
- net /BBB_p6: track 53.0 -> 47.4 mm
- net Net-(R21-Pad1): track 0.00 -> 4.47 mm
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Other:
- board text added: "Grupo de Controle - LNLS Vacuum BBB Controller versão 2.0 - Jul/2018"
- board text removed: "Grupo de Controle - LNLS Conversor USB/RS-485 versão 2.1 - Out/2016"
