File: hardware/kicad/VBC v2.0/VBC_v2-0.kicad_pcb (KiCad board)
At the start: 2 copper layers, 160 x 100.1 mm, 89 parts, among them J1 RJ11, J2 RJ11, J3 RJ11, J4 RJ11, J5 RJ25, J6 Conn_01x02, J7 Conn_01x01, J8 Conn_01x01, K1 RELAY_Metaltex, K2 RELAY_Metaltex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

Commit message: updated hardware version 2.0
Routing:
- net GND: track 409.2 -> 415.7 mm
Changed lines of the file:
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@@
     (thickness 1.6)
     (drawings 18)
-    (tracks 759)
+    (tracks 771)
     (zones 0)
     (modules 89)
@@
   )
   (setup
-    (last_trace_width 0.8)
+    (last_trace_width 0.4)
     (user_trace_width 0.01)
     (user_trace_width 0.25)
@@
   (segment (start 243.82208 47.9434) (end 243.82208 48.53012) (width 0.8) (layer F.Cu) (net 4))
   (segment (start 220.96208 96.90188) (end 220.96208 96.2034) (width 0.8) (layer F.Cu) (net 49))
+  (segment (start 163.62 113.29) (end 163.62 111.18) (width 0.4) (layer F.Cu) (net 68))
+  (segment (start 163.69 111.11) (end 163.69 111.1) (width 0.4) (layer F.Cu) (net 68))
+  (segment (start 163.62 111.18) (end 163.69 111.11) (width 0.4) (layer F.Cu) (net 68))
+  (segment (start 179.63 106.77) (end 179.63 106.89) (width 0.4) (layer F.Cu) (net 68))
+  (segment (start 179.98 107.99) (end 182.18 107.99) (width 0.4) (layer F.Cu) (net 68))
+  (segment (start 179.91 107.92) (end 179.98 107.99) (width 0.4) (layer F.Cu) (net 68))
+  (segment (start 179.91 107.17) (end 179.91 107.92) (width 0.4) (layer F.Cu) (net 68))
+  (segment (start 179.63 106.89) (end 179.91 107.17) (width 0.4) (layer F.Cu) (net 68))
+  (segment (start 179.63 106.5875) (end 179.63 106.77) (width 0.4) (layer F.Cu) (net 68))
+  (segment (start 179.63 106.77) (end 179.63 106.63) (width 0.4) (layer F.Cu) (net 68))
+  (segment (start 181.16 106.98) (end 182.28 105.86) (width 0.4) (layer F.Cu) (net 68))
+  (segment (start 179.98 106.98) (end 181.16 106.98) (width 0.4) (layer F.Cu) (net 68))
+  (segment (start 179.63 106.63) (end 179.98 106.98) (width 0.4) (layer F.Cu) (net 68))
   (segment (start 152.785 56.39) (end 152.785 54.045) (width 0.4) (layer F.Cu) (net 68))
   (segment (start 152.785 54.045) (end 152.44 53.7) (width 0.4) (layer F.Cu) (net 68))
@@
   (segment (start 179.74 108.125) (end 179.74 107.17) (width 0.4) (layer F.Cu) (net 68))
   (segment (start 178.0525 106.5875) (end 179.1575 106.5875) (width 0.4) (layer F.Cu) (net 68))
-  (segment (start 179.1575 106.5875) (end 181.3225 106.5875) (width 0.4) (layer F.Cu) (net 68))
-  (segment (start 181.3225 106.5875) (end 182.05 105.86) (width 0.4) (layer F.Cu) (net 68))
-  (segment (start 184 105.86) (end 182.05 105.86) (width 0.4) (layer F.Cu) (net 68))
+  (segment (start 179.1575 106.5875) (end 179.63 106.5875) (width 0.4) (layer F.Cu) (net 68))
+  (segment (start 184 105.86) (end 182.28 105.86) (width 0.4) (layer F.Cu) (net 68))
   (segment (start 178.0525 103.9875) (end 176.1425 103.9875) (width 0.4) (layer F.Cu) (net 68))
   (segment (start 176.1425 103.9875) (end 176.0825 103.9875) (width 0.4) (layer F.Cu) (net 68))

Commit message: updated hardware version 2.0
Connections:
- J7 pad 2: (no net) -> GND
Routing:
- net GND: track 415.7 -> 294.2 mm
Changed lines of the file:
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@@
 (kicad_pcb (version 4) (host pcbnew 4.0.7-e2-6376~58~ubuntu16.04.1)
   (general
-    (links 210)
+    (links 211)
     (no_connects 0)
     (area 98.01079 28.702 282.749801 146.050001)
     (thickness 1.6)
     (drawings 18)
-    (tracks 771)
+    (tracks 761)
     (zones 0)
     (modules 89)
@@
     (mod_text_size 1 1)
     (mod_text_width 0.15)
-    (pad_size 1.59 1.59)
-    (pad_drill 0.89)
+    (pad_size 7 7)
+    (pad_drill 3)
     (pad_to_mask_clearance 0.2)
     (aux_axis_origin 0 0)
@@
     (pad 1 thru_hole circle (at 25.25 14.65 180) (size 7 7) (drill 3) (layers *.Cu *.Mask)
       (net 68 GND))
-    (pad 2 thru_hole circle (at 25.25 53.75 180) (size 7 7) (drill 3) (layers *.Cu *.Mask))
+    (pad 2 thru_hole circle (at 25.25 53.75 180) (size 7 7) (drill 3) (layers *.Cu *.Mask)
+      (net 68 GND))
   )
   (module Pin_Headers:Pin_Header_Straight_2x06_Pitch2.54mm (layer F.Cu)
@@
   (segment (start 152.785 56.39) (end 152.785 54.045) (width 0.4) (layer F.Cu) (net 68))
   (segment (start 152.785 54.045) (end 152.44 53.7) (width 0.4) (layer F.Cu) (net 68))
-  (segment (start 152.785 56.39) (end 152.785 59.355) (width 0.4) (layer F.Cu) (net 68))
-  (segment (start 152.785 59.355) (end 160.82 67.39) (width 0.4) (layer F.Cu) (net 68))
   (segment (start 268.86148 100.18) (end 268.7532 100.18) (width 1) (layer F.Cu) (net 68))
   (segment (start 116.57 124.51) (end 152.63 124.51) (width 0.8) (layer B.Cu) (net 68))
@@
   (segment (start 176.7275 103.3375) (end 176.5025 103.5625) (width 0.25) (layer F.Cu) (net 68))
   (segment (start 167.5275 105.9375) (end 167.5025 105.9625) (width 0.25) (layer F.Cu) (net 68))
-  (segment (start 160.82 67.39) (end 160.82 78.23) (width 0.4) (layer F.Cu) (net 68))
   (segment (start 154.59 122.55) (end 152.63 124.51) (width 0.8) (layer B.Cu) (net 68))
   (segment (start 152.63 124.51) (end 166.12 124.51) (width 0.8) (layer B.Cu) (net 68))
@@
   (segment (start 173.61 83.19) (end 183.01 92.59) (width 0.8) (layer B.Cu) (net 68))
   (segment (start 173.61 45.59) (end 173.61 83.19) (width 0.8) (layer B.Cu) (net 68))
-  (segment (start 160.82 78.23) (end 148.64 90.41) (width 0.4) (layer F.Cu) (net 68))
-  (segment (start 148.64 90.41) (end 132.55 90.41) (width 0.4) (layer F.Cu) (net 68))
-  (segment (start 132.55 90.41) (end 122.86 100.1) (width 0.4) (layer F.Cu) (net 68))
-  (segment (start 122.86 100.1) (end 122.86 112.28) (width 0.4) (layer F.Cu) (net 68))
-  (segment (start 122.86 112.28) (end 130.4 119.82) (width 0.4) (layer F.Cu) (net 68))
-  (segment (start 130.4 119.82) (end 149.17 119.82) (width 0.4) (layer F.Cu) (net 68))
-  (segment (start 149.17 119.82) (end 154.59 114.4) (width 0.4) (layer F.Cu) (net 68))
   (segment (start 154.59 114.4) (end 154.59 122.55) (width 0.8) (layer B.Cu) (net 68))
   (segment (start 266.9748 68.6755) (end 260.6045 68.6755) (width 1) (layer F.Cu) (net 69))

Commit message: updated hardware version 2.0
Parts:
- P2: moved to B.Cu
- moved REF** 6.00 mm to (122.6, 129.6)
- moved P2 3.57 mm to (184.7, 114.7), turned to 180 degrees
- moved D13 1.90 mm to (115.9, 75.2)
- moved D14 1.90 mm to (115.9, 69.1)
- moved SW1 1.89 mm to (117.4, 116.4)
- moved P3 1.50 mm to (117.9, 87.1)
- moved P4 1.50 mm to (117.9, 104.1)
Routing:
- net GND: track 294.2 -> 325.5 mm, vias 5 -> 6
- net /USB_converter_485./RS485-: track 73.5 -> 89.2 mm
- net Net-(R31-Pad2): track 22.8 -> 34.5 mm
- net /USB_converter_485./RS485+: track 112.0 -> 102.5 mm
- net Net-(C4-Pad1): track 49.9 -> 42.8 mm
- net +24V: track 323.6 -> 318.5 mm
- net /USB_converter_485./USB_D-: track 21.6 -> 16.9 mm
- net Net-(R30-Pad2): track 29.1 -> 32.6 mm
- net Net-(D14-Pad2): track 21.8 -> 24.1 mm
- net Net-(D13-Pad2): track 22.7 -> 24.9 mm
- net /USB_converter_485./TXLED#: track 80.4 -> 82.5 mm
- net /USB_converter_485./RXLED#: track 87.5 -> 89.5 mm
- net /USB_converter_485./5V_ISOLATED: track 142.7 -> 144.7 mm
- net /USB_converter_485./USB_D+: track 19.0 -> 19.9 mm

Commit message: updated hardware version 2.0
Parts:
- D13, D14, P3, P4, REF**, SW1: moved to B.Cu
- moved REF** 5.09 mm to (121.8, 124.6)
- turned D13 to 90 degrees
- turned D14 to 90 degrees
- turned P3 to 90 degrees
- turned P4 to 90 degrees
- turned SW1 to 270 degrees
Routing:
- net GND: track 325.5 -> 290.2 mm
- net /USB_converter_485./TXLED#: track 82.5 -> 100.0 mm
- net /USB_converter_485./RXLED#: track 89.5 -> 104.0 mm
- net Net-(R31-Pad2): track 34.5 -> 22.6 mm
- net /USB_converter_485./RS485+: track 102.5 -> 91.2 mm
- net +24V: track 318.5 -> 311.0 mm
- net /USB_converter_485./RS485-: track 89.2 -> 85.9 mm
- net /USB_converter_485./5V_ISOLATED: track 144.7 -> 143.1 mm
- net Net-(R30-Pad2): track 32.6 -> 33.9 mm
- net Net-(D14-Pad2): track 24.1 -> 23.0 mm, vias 1 -> 0
- net Net-(D13-Pad2): track 24.9 -> 24.4 mm, vias 1 -> 0

Commit message: updated hardware version 2.0
Parts:
- ?: renamed from Beagle1; value BeagleBone -> (none)
- ?: renamed from J8; value Conn_01x01 -> (none)
- C1: value Conn_SMA_90graus -> (none)
- J6: value Conn_01x02 -> (none)
- REF**: value Pin_Header_Angled_1x02_Pitch2.54mm -> (none)
- moved G*** 8.49 mm to (248.8, 109.3)
Routing:
- net Net-(K2-Pad11): track 1.49 -> 0.00 mm
- net GND: track 290.2 -> 288.7 mm
Other:
- board text added: "GND"
- board text added: "Grupo de Controle - LNLS Vacuum BBB Controller Patrícia Nallin Rafael Ito Júlia Giatti versão 2.0 - Jul/2018"
- board text added: "P8"
- board text added: "P9"
- board text added: "VCC"
- board text removed: "Grupo de Controle - LNLS Vacuum BBB Controller versão 2.0 - Jul/2018"

Commit message: updated hardware version 2.0
Other:
- board text added: "Grupo de Controle - LNLS Vacuum BBB Controller Júlia Giatti Patrícia Nallin Rafael Ito versão 2.0 - Jul/2018"
- board text removed: "Grupo de Controle - LNLS Vacuum BBB Controller Patrícia Nallin Rafael Ito Júlia Giatti versão 2.0 - Jul/2018"
Changed lines of the file:
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@@
   (page A4)
   (title_block
-    (title "Conversor USB/RS-485")
+    (title "Vacuum BBB Controler")
     (date 2016-02-02)
     (rev 1)
     (company "Laboratório Nacional de Luz Síncrotron / Grupo de Controle")
-    (comment 2 ?)
-    (comment 3 "Eduardo Pereira Coelho")
   )
   (layers
@@
   )
   (setup
-    (last_trace_width 0.8)
+    (last_trace_width 0.4)
     (user_trace_width 0.01)
     (user_trace_width 0.25)
@@
   (gr_line (start 273.45148 37.28028) (end 273.45148 137.28028) (angle 90) (layer Edge.Cuts) (width 0.15))
   (gr_line (start 144.4598 37.28028) (end 273.45148 37.28028) (angle 90) (layer Edge.Cuts) (width 0.15))
-  (gr_text "Grupo de Controle - LNLS\nVacuum BBB Controller\nPatrícia Nallin\nRafael Ito\nJúlia Giatti\nversão 2.0 - Jul/2018" (at 246.66 125.12) (layer F.SilkS)
+  (gr_text "Grupo de Controle - LNLS\nVacuum BBB Controller\nJúlia Giatti\nPatrícia Nallin\nRafael Ito\nversão 2.0 - Jul/2018" (at 246.66 125.12) (layer F.SilkS)
     (effects (font (size 1.2 1.2) (thickness 0.2)))
   )
