File: hardware/kicad/VBC v2.0/VBC_v2-0.sch (KiCad schematic (older format))
At the start: 55 parts, among them J1 RJ11, J2 RJ11, J3 RJ11, J4 RJ11, J5 RJ25, J6 Conn_01x02, J7 Conn_01x01, J8 Conn_01x01, K1 RELAY_Metaltex, K2 RELAY_Metaltex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

Commit message: new hardware version - v2.0
Parts:
- added R34: 5k, Resistors_SMD:R_0805_HandSoldering, symbol R
- added R35: 10k, Resistors_SMD:R_0805_HandSoldering, symbol R
Connections:
- net at R21.1: now also R35.2; no longer C1.1
- new net: C1.1, R34.1
- new net: R34.2, R35.1
Other:
- moved on the sheet: C1, R21, R22
Changed lines of the file:
@@
 L R R21
 U 1 1 5B4DFA8E
-P 7135 3295
-F 0 "R21" V 7215 3295 50  0000 C CNN
-F 1 "10k" V 7135 3295 50  0000 C CNN
-F 2 "Resistors_SMD:R_0805_HandSoldering" V 7065 3295 50  0001 C CNN
-F 3 "" H 7135 3295 50  0001 C CNN
-	1    7135 3295
+P 7080 3470
+F 0 "R21" V 7160 3470 50  0000 C CNN
+F 1 "10k" V 7080 3470 50  0000 C CNN
+F 2 "Resistors_SMD:R_0805_HandSoldering" V 7010 3470 50  0001 C CNN
+F 3 "" H 7080 3470 50  0001 C CNN
+	1    7080 3470
 	1    0    0    -1
 $EndComp
@@
 L R R22
 U 1 1 5B4DFA8F
-P 7135 3750
-F 0 "R22" V 7215 3750 50  0000 C CNN
-F 1 "5k" V 7135 3750 50  0000 C CNN
-F 2 "Resistors_SMD:R_0805_HandSoldering" V 7065 3750 50  0001 C CNN
-F 3 "" H 7135 3750 50  0001 C CNN
-	1    7135 3750
+P 7080 3925
+F 0 "R22" V 7160 3925 50  0000 C CNN
+F 1 "5k" V 7080 3925 50  0000 C CNN
+F 2 "Resistors_SMD:R_0805_HandSoldering" V 7010 3925 50  0001 C CNN
+F 3 "" H 7080 3925 50  0001 C CNN
+	1    7080 3925
 	1    0    0    -1
 $EndComp
@@
 L GND #PWR09
 U 1 1 5B4DFA90
-P 7135 3985
-F 0 "#PWR09" H 7135 3735 50  0001 C CNN
-F 1 "GND" H 7135 3835 50  0000 C CNN
-F 2 "" H 7135 3985 50  0001 C CNN
-F 3 "" H 7135 3985 50  0001 C CNN
-	1    7135 3985
-	1    0    0    -1
-$EndComp
-Text Label 7420 3520 0    60   ~ 0
+P 7080 4075
+F 0 "#PWR09" H 7080 3825 50  0001 C CNN
+F 1 "GND" H 7080 3925 50  0000 C CNN
+F 2 "" H 7080 4075 50  0001 C CNN
+F 3 "" H 7080 4075 50  0001 C CNN
+	1    7080 4075
+	1    0    0    -1
+$EndComp
+Text Label 7365 3695 0    60   ~ 0
 AIn_BBB
 $Comp
 L Conn_SMA_90graus C1
 U 1 1 5B4DFA91
-P 7135 2945
-F 0 "C1" H 7230 2825 60  0000 C CNN
-F 1 "Conn_SMA_90graus" H 7135 3075 60  0000 C CNN
-F 2 "Connectors:SMA_THT_Jack_Straight" H 7135 2945 60  0001 C CNN
-F 3 "" H 7135 2945 60  0000 C CNN
-	1    7135 2945
-	0    -1   -1   0
+P 7485 2620
+F 0 "C1" H 7580 2500 60  0000 C CNN
+F 1 "Conn_SMA_90graus" H 7485 2750 60  0000 C CNN
+F 2 "Connectors:SMA_THT_Jack_Straight" H 7485 2620 60  0001 C CNN
+F 3 "" H 7485 2620 60  0000 C CNN
+	1    7485 2620
+	1    0    0    -1
 $EndComp
 $Comp
 L GND #PWR010
 U 1 1 5B4DFA93
-P 7405 2945
-F 0 "#PWR010" H 7405 2695 50  0001 C CNN
-F 1 "GND" H 7405 2795 50  0000 C CNN
-F 2 "" H 7405 2945 50  0001 C CNN
-F 3 "" H 7405 2945 50  0001 C CNN
-	1    7405 2945
-	0    -1   -1   0
+P 7485 2890
+F 0 "#PWR010" H 7485 2640 50  0001 C CNN
+F 1 "GND" H 7485 2740 50  0000 C CNN
+F 2 "" H 7485 2890 50  0001 C CNN
+F 3 "" H 7485 2890 50  0001 C CNN
+	1    7485 2890
+	1    0    0    -1
 $EndComp
 $Comp
@@
 F1 "USB_converter_485.sch" 60
 $EndSheet
+$Comp
+L R R35
+U 1 1 5B4FA405
+P 7080 3120
+F 0 "R35" V 7160 3120 50  0000 C CNN
+F 1 "10k" V 7080 3120 50  0000 C CNN
+F 2 "Resistors_SMD:R_0805_HandSoldering" V 7010 3120 50  0001 C CNN
+F 3 "" H 7080 3120 50  0001 C CNN
+	1    7080 3120
+	1    0    0    -1
+$EndComp
+$Comp
+L R R34
+U 1 1 5B4FA571
+P 7080 2765
+F 0 "R34" V 7160 2765 50  0000 C CNN
+F 1 "5k" V 7080 2765 50  0000 C CNN
+F 2 "Resistors_SMD:R_0805_HandSoldering" V 7010 2765 50  0001 C CNN
+F 3 "" H 7080 2765 50  0001 C CNN
+	1    7080 2765
+	1    0    0    -1
+$EndComp
 Connection ~ 3090 6090
 Wire Wire Line
@@
 	1345 5250 1430 5250
 Wire Wire Line
-	7135 3445 7135 3600
-Wire Wire Line
-	7135 3520 7420 3520
-Connection ~ 7135 3520
-Wire Wire Line
-	7135 3985 7135 3900
+	7080 3620 7080 3775
+Wire Wire Line
+	7080 3695 7365 3695
+Connection ~ 7080 3695
 Wire Wire Line
 	7085 4795 7085 4760
@@
 Wire Wire Line
 	10715 4180 10715 4135
+Wire Wire Line
+	7080 3320 7080 3270
+Wire Wire Line
+	7080 2970 7080 2915
+Wire Wire Line
+	7080 2615 7285 2615
+Wire Wire Line
+	7285 2615 7285 2620
 $EndSCHEMATC
