File: hardware/kicad/VBC v2.1/VBC_v2-1.kicad_pcb (KiCad board)
At the start: 2 copper layers, 160 x 100.1 mm, 89 parts, among them J1 RJ11, J2 RJ11, J3 RJ11, J4 RJ11, J5 RJ25, J7 Conn_01x01, K1 RELAY_Metaltex, K2 RELAY_Metaltex, K3 RELAY_Metaltex, K4 RELAY_Metaltex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

Commit message: added VBC v2.2 files
Other:
- board text added: "Grupo de Controle - LNLS Vacuum BBB Controller Júlia Giatti Patrícia Nallin Rafael Ito versão 2.1 - Jul/2018"
- board text removed: "Grupo de Controle - LNLS Vacuum BBB Controller Júlia Giatti Patrícia Nallin Rafael Ito versão 2.0 - Jul/2018"
Changed lines of the file:
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@@
-(kicad_pcb (version 4) (host pcbnew 4.0.7-e2-6376~58~ubuntu16.04.1)
+(kicad_pcb (version 4) (host pcbnew 4.0.7-e2-6376~61~ubuntu18.04.1)
   (general
     (links 211)
@@
   )
   (layers
-    (0 F.Cu signal)
-    (31 B.Cu signal)
+    (0 F.Cu signal hide)
+    (31 B.Cu signal hide)
     (32 B.Adhes user)
     (33 F.Adhes user)
@@
   )
   (setup
-    (last_trace_width 0.8)
+    (last_trace_width 0.4)
     (user_trace_width 0.01)
     (user_trace_width 0.25)
@@
     (fp_line (start -1.45 -1.55) (end 9.07 -1.55) (layer F.CrtYd) (width 0.05))
     (fp_line (start 9.07 -1.55) (end 9.07 19.33) (layer F.CrtYd) (width 0.05))
-    (fp_text user %R (at 3.94 9.16 180) (layer F.Fab)
+    (fp_text user %R (at 3.94 9.16 180) (layer F.SilkS)
       (effects (font (size 1 1) (thickness 0.15)))
     )
@@
     (fp_line (start -1.45 -1.55) (end 9.07 -1.55) (layer F.CrtYd) (width 0.05))
     (fp_line (start 9.07 -1.55) (end 9.07 19.33) (layer F.CrtYd) (width 0.05))
-    (fp_text user %R (at 3.94 9.16 180) (layer F.Fab)
+    (fp_text user %R (at 3.94 9.16 180) (layer F.SilkS)
       (effects (font (size 1 1) (thickness 0.15)))
     )
@@
     (fp_line (start -1.45 -1.55) (end 9.07 -1.55) (layer F.CrtYd) (width 0.05))
     (fp_line (start 9.07 -1.55) (end 9.07 19.33) (layer F.CrtYd) (width 0.05))
-    (fp_text user %R (at 3.94 9.16 180) (layer F.Fab)
+    (fp_text user %R (at 3.94 9.16 180) (layer F.SilkS)
       (effects (font (size 1 1) (thickness 0.15)))
     )
@@
     (fp_line (start -1.45 -1.55) (end 9.07 -1.55) (layer F.CrtYd) (width 0.05))
     (fp_line (start 9.07 -1.55) (end 9.07 19.33) (layer F.CrtYd) (width 0.05))
-    (fp_text user %R (at 3.94 9.16 180) (layer F.Fab)
+    (fp_text user %R (at 3.94 9.16 180) (layer F.SilkS)
       (effects (font (size 1 1) (thickness 0.15)))
     )
@@
       (effects (font (size 1 1) (thickness 0.15)) (justify mirror))
     )
-    (fp_text value BC817 (at 0 -2.5 90) (layer B.Fab)
+    (fp_text value BC817 (at 0 -2.5 90) (layer B.SilkS)
       (effects (font (size 1 1) (thickness 0.15)) (justify mirror))
     )
@@
       (effects (font (size 1 1) (thickness 0.15)) (justify mirror))
     )
-    (fp_text value 1k (at 0 -1.75 270) (layer B.Fab)
+    (fp_text value 1k (at 0 -1.75 270) (layer B.SilkS)
       (effects (font (size 1 1) (thickness 0.15)) (justify mirror))
     )
@@
       (effects (font (size 1 1) (thickness 0.15)) (justify mirror))
     )
-    (fp_text value 1k (at 0 -1.75 180) (layer B.Fab)
+    (fp_text value 1k (at 0 -1.75 180) (layer B.SilkS)
       (effects (font (size 1 1) (thickness 0.15)) (justify mirror))
     )
@@
       (effects (font (size 1 1) (thickness 0.15)))
     )
-    (fp_text value 10k (at 0 1.75 270) (layer F.Fab)
+    (fp_text value 10k (at 0 1.75 270) (layer F.SilkS)
       (effects (font (size 1 1) (thickness 0.15)))
     )
@@
       (effects (font (size 1 1) (thickness 0.15)))
     )
-    (fp_text value 5k (at 0 1.75 270) (layer F.Fab)
+    (fp_text value 5k (at 0 1.75 270) (layer F.SilkS)
       (effects (font (size 1 1) (thickness 0.15)))
     )
@@
     (tags "capacitor 0805")
     (attr smd)
-    (fp_text reference C9 (at -3.97 -0.49 90) (layer F.SilkS)
+    (fp_text reference C9 (at 3.4125 -0.6025 90) (layer F.SilkS)
       (effects (font (size 0.7 0.7) (thickness 0.1)))
     )
-    (fp_text value 47nF (at -3.95 0.65 90) (layer F.SilkS)
+    (fp_text value 47nF (at 3.8875 0.3725 90) (layer F.SilkS)
       (effects (font (size 0.7 0.7) (thickness 0.1)))
     )
@@
       (effects (font (size 1 1) (thickness 0.15)))
     )
-    (fp_text value 5k (at 0 1.75 180) (layer F.Fab)
+    (fp_text value 5k (at 0 1.75 180) (layer F.SilkS)
       (effects (font (size 1 1) (thickness 0.15)))
     )
@@
       (effects (font (size 1 1) (thickness 0.15)))
     )
-    (fp_text value 10k (at 0 1.75 180) (layer F.Fab)
+    (fp_text value 10k (at 0 1.75 180) (layer F.SilkS)
       (effects (font (size 1 1) (thickness 0.15)))
     )
@@
   (gr_line (start 273.45148 37.28028) (end 273.45148 137.28028) (angle 90) (layer Edge.Cuts) (width 0.15))
   (gr_line (start 144.4598 37.28028) (end 273.45148 37.28028) (angle 90) (layer Edge.Cuts) (width 0.15))
-  (gr_text "Grupo de Controle - LNLS\nVacuum BBB Controller\nJúlia Giatti\nPatrícia Nallin\nRafael Ito\nversão 2.0 - Jul/2018" (at 246.66 125.12) (layer F.SilkS)
+  (gr_text "Grupo de Controle - LNLS\nVacuum BBB Controller\nJúlia Giatti\nPatrícia Nallin\nRafael Ito\nversão 2.1 - Jul/2018" (at 246.66 125.12) (layer F.SilkS)
     (effects (font (size 1.2 1.2) (thickness 0.2)))
   )
@@
   (segment (start 226.75 82.4) (end 221.225 82.4) (width 0.8) (layer B.Cu) (net 81))
   (segment (start 227.4962 81.6538) (end 226.75 82.4) (width 0.8) (layer B.Cu) (net 81))
-  (segment (start 250.075 53.3) (end 250.075 54.8) (width 0.8) (layer F.Cu) (net 82) (status 400000))
+  (segment (start 250.075 53.3) (end 250.075 54.8) (width 0.8) (layer F.Cu) (net 82))
   (segment (start 250.075 54.8) (end 252.125 56.85) (width 0.8) (layer F.Cu) (net 82))
-  (segment (start 258.89446 56.85) (end 260.07522 55.66924) (width 0.8) (layer F.Cu) (net 82) (status 800000))
+  (segment (start 258.89446 56.85) (end 260.07522 55.66924) (width 0.8) (layer F.Cu) (net 82))
   (segment (start 252.125 56.85) (end 258.89446 56.85) (width 0.8) (layer F.Cu) (net 82))
   (segment (start 238.74208 47.9434) (end 238.74208 51.44208) (width 0.8) (layer F.Cu) (net 82))
@@
   (segment (start 217.561 74.207) (end 217.561 76.16356) (width 0.8) (layer B.Cu) (net 87))
   (segment (start 217.561 76.16356) (end 218.78782 77.39038) (width 0.8) (layer B.Cu) (net 87))
-  (segment (start 262.61522 56.93924) (end 262.61522 58.78478) (width 0.8) (layer F.Cu) (net 91) (status 400000))
+  (segment (start 262.61522 56.93924) (end 262.61522 58.78478) (width 0.8) (layer F.Cu) (net 91))
   (segment (start 260.52 60.88) (end 255.34 60.88) (width 0.8) (layer F.Cu) (net 91))
   (segment (start 262.61522 58.78478) (end 260.52 60.88) (width 0.8) (layer F.Cu) (net 91))
-  (segment (start 261.875 50.19638) (end 260.46808 50.19638) (width 0.8) (layer F.Cu) (net 91) (status 800000))
-  (segment (start 260.46808 50.19638) (end 260.07522 50.58924) (width 0.8) (layer F.Cu) (net 91) (status C00000))
+  (segment (start 261.875 50.19638) (end 260.46808 50.19638) (width 0.8) (layer F.Cu) (net 91))
+  (segment (start 260.46808 50.19638) (end 260.07522 50.58924) (width 0.8) (layer F.Cu) (net 91))
   (segment (start 255.34 60.88) (end 255.34 72.72968) (width 0.8) (layer B.Cu) (net 91))
   (segment (start 252.3082 75.7564) (end 269.29572 75.7564) (width 0.8) (layer F.Cu) (net 91))
