File: hardware/kicad/VBC v2.1/VBC_v2-1.sch (KiCad schematic (older format))
At the start: 57 parts, among them J1 RJ11, J2 RJ11, J3 RJ11, J4 RJ11, J5 RJ25, J6 Conn_01x02, J7 Conn_01x01, J8 Conn_01x01, K1 RELAY_Metaltex, K2 RELAY_Metaltex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

Commit message: added VBC v2.2 files
Parts:
- renumbered J4 to J1, J1 to J4, K4 to K1, K1 to K4
Connections:
- net +24V: no longer K4.13 (C2), K4.4 (C1)
- net BBB_p1: now also Beagle1.C12 (B12), R4.1; no longer Beagle1.B18, R1.1
- net BBB_p4: now also Beagle1.B18, R1.1; no longer Beagle1.C12 (B12), R4.1
- new net: K4.13 (C2), K4.4 (C1)
- no-connect marks 84 -> 82
